File: splitnsnap.kicad_sch (KiCad schematic)
At the start: 0 parts

Commit message: things
Other:
- sheet left: file side.kicad_sch -> left.kicad_sch
- sheet right: file side.kicad_sch -> right.kicad_sch
Changed lines of the file:
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@@
 	(paper "A4")
 	(sheet
-		(at 71.12 48.26)
-		(size 23.495 13.335)
+		(at 74.295 52.705)
+		(size 15.875 10.16)
 		(exclude_from_sim no)
 		(in_bom yes)
@@
 		)
 		(property "Sheetname" "left"
-			(at 71.12 47.5484 0)
+			(at 74.295 51.9934 0)
 			(show_name no)
 			(do_not_autoplace no)
@@
 			)
 		)
-		(property "Sheetfile" "side.kicad_sch"
-			(at 71.12 62.1796 0)
+		(property "Sheetfile" "left.kicad_sch"
+			(at 74.295 63.4496 0)
 			(show_name no)
 			(do_not_autoplace no)
@@
 	)
 	(sheet
-		(at 38.1 48.26)
-		(size 23.495 13.335)
+		(at 49.53 52.705)
+		(size 15.875 10.16)
 		(exclude_from_sim no)
 		(in_bom yes)
 		(on_board yes)
 		(dnp no)
-		(fields_autoplaced yes)
 		(stroke
 			(width 0.1524)
@@
 		)
 		(property "Sheetname" "right"
-			(at 38.1 47.5484 0)
+			(at 49.53 51.9934 0)
 			(show_name no)
 			(do_not_autoplace no)
@@
 			)
 		)
-		(property "Sheetfile" "side.kicad_sch"
-			(at 38.1 62.1796 0)
+		(property "Sheetfile" "right.kicad_sch"
+			(at 49.53 63.4496 0)
 			(show_name no)
 			(do_not_autoplace no)
